File: Choc2.kicad_pcb (KiCad board)
At the start: 2 copper layers, 40 x 100 mm, 19 parts, among them J1 Conn_01x02, J4 Conn_01x03, SW1 SW_PUSH, SW2 SW_PUSH, SW3 SW_PUSH, SW4 SW_PUSH, SW5 SW_PUSH, SW6 SW_PUSH, SW7 SW_PUSH, U1 xiao-th

Commit message: XH
Parts:
- J1: footprint Connector_JST:JST_PH_S2B-PH-K_1x02_P2.00mm_Horizontal -> Connector_JST:JST_XH_S2B-XH-A_1x02_P2.50mm_Horizontal
- J4: footprint Connector_JST:JST_PH_S3B-PH-K_1x03_P2.00mm_Horizontal -> Connector_JST:JST_XH_S3B-XH-A_1x03_P2.50mm_Horizontal
- moved J1 3.58 mm to (54.0, 65.8)
- moved J4 3.50 mm to (86.0, 62.0)
Routing:
- net VCC: track 217.1 -> 223.6 mm
- net LED2: track 25.2 -> 28.9 mm
