File: Choc2.kicad_pcb (KiCad board)
At the start: 2 copper layers, 40 x 100 mm, 19 parts, among them J1 Conn_01x02, J4 Conn_01x03, SW1 SW_PUSH, SW2 SW_PUSH, SW3 SW_PUSH, SW4 SW_PUSH, SW5 SW_PUSH, SW6 SW_PUSH, SW7 SW_PUSH, U1 xiao-th

Commit message: Remap
Parts:
- OL1: footprint 07:MODULE_DM-OLED096-636 -> 07:MODULE_DM-OLED096-636_3D
- moved LED7 47.6 mm to (62.0, 88.0)
- moved SW7 47.2 mm to (62.0, 96.0)
- moved LED5 25.5 mm to (61.0, 132.0)
- moved SW4 25.5 mm to (79.0, 140.0)
- moved SW5 25.5 mm to (61.0, 140.0)
- moved LED4 25.4 mm to (79.0, 132.0)
- moved LED6 18.1 mm to (61.0, 114.0)
- moved LED3 18.0 mm to (79.0, 114.0)
- moved SW3 18.0 mm to (79.0, 122.0)
- moved SW6 18.0 mm to (61.0, 122.0)
- moved LED1 17.9 mm to (78.0, 80.0)
- moved SW1 17.9 mm to (78.0, 88.0)
- moved LED2 16.0 mm to (78.0, 96.0)
- moved SW2 16.0 mm to (78.0, 104.0)
Connections:
- LED5 pad 2: unconnected-(LED5-DOUT-Pad2) -> Net-(LED5-DOUT)
- LED6 pad 2: unconnected-(LED6-DOUT-Pad2) -> Net-(LED6-DOUT)
- LED6 pad 4: unconnected-(LED5-DOUT-Pad2) -> Net-(LED5-DOUT)
- LED7 pad 4: unconnected-(LED6-DOUT-Pad2) -> Net-(LED6-DOUT)
- U1 pad 1: SW4 -> SW1
- U1 pad 10: SW2 -> SCL
- U1 pad 11: SW7 -> LED2
- U1 pad 2: SW3 -> SW2
- U1 pad 3: SW5 -> SW3
- U1 pad 4: SW6 -> SW4
- U1 pad 5: SDA -> LED
- U1 pad 6: SCL -> SW5
- U1 pad 7: LED -> SW6
- U1 pad 8: SW1 -> SW7
- U1 pad 9: LED2 -> SDA
Routing:
- net SW7: track 138.8 -> 46.6 mm
- net Net-(LED5-DOUT): track 0.00 -> 47.2 mm
- net Net-(LED6-DOUT): track 0.00 -> 39.3 mm
- net unconnected-(LED5-DOUT-Pad2): track 33.8 -> 0.00 mm
- net SW1: track 57.0 -> 25.2 mm, vias 2 -> 0
- net SW4: track 57.5 -> 80.7 mm
- net SW6: track 79.2 -> 59.3 mm, vias 1 -> 0
- net SCL: track 24.2 -> 4.41 mm
- net SW3: track 42.3 -> 60.6 mm, vias 0 -> 1
- net SW5: track 67.7 -> 83.1 mm, vias 0 -> 2
- net SDA: track 19.6 -> 4.41 mm
- net unconnected-(LED6-DOUT-Pad2): track 13.4 -> 0.00 mm, vias 2 -> 0
- net Net-(LED3-DOUT): track 31.2 -> 19.1 mm
- net GND: track 32.8 -> 42.9 mm, vias 14 -> 13
- net VCC: track 216.9 -> 209.7 mm
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