File: Choc2.kicad_sch (KiCad schematic)
At the start: 19 parts, among them J1 Conn_01x02, J4 Conn_01x03, SW1 SW_PUSH, SW2 SW_PUSH, SW3 SW_PUSH, SW4 SW_PUSH, SW5 SW_PUSH, SW6 SW_PUSH, SW7 SW_PUSH, U1 xiao-th

Commit message: chipSocket
Connections:
- net GND: now also OL1.4 (GND); no longer OL1.1 (SDA)
- net SCL: now also OL1.2 (SCL); no longer OL1.3 (VCC)
- net SDA: now also OL1.1 (SDA); no longer OL1.4 (GND)
- net VCC: now also OL1.3 (VCC); no longer OL1.2 (SCL)

Commit message: XH
Parts:
- J1: footprint Connector_JST:JST_PH_S2B-PH-K_1x02_P2.00mm_Horizontal -> Connector_JST:JST_XH_S2B-XH-A_1x02_P2.50mm_Horizontal
- J4: footprint Connector_JST:JST_PH_S3B-PH-K_1x03_P2.00mm_Horizontal -> Connector_JST:JST_XH_S3B-XH-A_1x03_P2.50mm_Horizontal
