File: Choc2.kicad_sch (KiCad schematic)
At the start: 19 parts, among them J1 Conn_01x02, J4 Conn_01x03, SW1 SW_PUSH, SW2 SW_PUSH, SW3 SW_PUSH, SW4 SW_PUSH, SW5 SW_PUSH, SW6 SW_PUSH, SW7 SW_PUSH, U1 xiao-th

Commit message: Remap
Connections:
- net GND: now also OL1.1 (GND); no longer OL1.4 (GND)
- net LED: now also U1.5 (IO22_SDA); no longer U1.7 (IO16_TX)
- net LED2: now also U1.11 (IO18_MOSI); no longer U1.9 (IO19_SCK)
- net SCL: now also OL1.3 (SCL), U1.10 (IO20_MISO); no longer OL1.2 (SCL), U1.6 (IO23_SCL)
- net SDA: now also OL1.4 (SDA), U1.9 (IO19_SCK); no longer OL1.1 (SDA), U1.5 (IO22_SDA)
- net SW1: now also U1.1 (LP_A_IO0); no longer U1.8 (IO17_RX)
- net SW2: now also U1.2 (LP_A_IO1); no longer U1.10 (IO20_MISO)
- net SW3: now also U1.3 (LP_A_IO2); no longer U1.2 (LP_A_IO1)
- net SW4: now also U1.4 (IO21); no longer U1.1 (LP_A_IO0)
- net SW5: now also U1.6 (IO23_SCL); no longer U1.3 (LP_A_IO2)
- net SW6: now also U1.7 (IO16_TX); no longer U1.4 (IO21)
- net SW7: now also U1.8 (IO17_RX); no longer U1.11 (IO18_MOSI)
- net VCC: now also OL1.2 (VCC); no longer OL1.3 (VCC)
- no-connect marks 4 -> 2
Other:
- moved on the sheet: SW1, SW2, SW3, SW4, SW5, SW6, SW7
